File: pcb/USB Switch PCB.brd (EAGLE design)
At the start: 100 x 80 mm, 18 parts, among them Q1 2N7002P, Q2 2N7002P, U1 D1MINI, X1 AMPHENOL-0001LF, X2 UE27-USBA

Commit message: Auto-routed PCB with lots of nice stuff.
Parts:
- LED1: value GREEN -> ACT
- LED2: value RED -> PWR
- moved S1 58.5 mm to (15.2, 57.1), turned to 180 degrees
- moved R3 38.9 mm to (1.27, 7.62), turned to 90 degrees
- moved R4 38.7 mm to (24.1, 7.62), turned to 90 degrees
- moved Q1 33.0 mm to (15.2, 47.0)
- moved D1 32.7 mm to (15.2, 52.1)
- moved D2 31.8 mm to (10.2, 52.1)
- moved Q2 31.8 mm to (10.2, 47.0)
- moved LED2 19.1 mm to (3.81, 3.81), turned to 180 degrees
- moved R2 15.9 mm to (3.81, 7.62), turned to 90 degrees
- moved U1 14.5 mm to (1.27, 19.1)
- moved U$1 14.2 mm to (21.6, 55.9), turned to 180 degrees
- moved U$2 12.8 mm to (3.81, 55.9), turned to 180 degrees
- moved R1 7.62 mm to (21.6, 7.62), turned to 270 degrees
- moved X2 4.02 mm to (12.7, 66.0)
- moved LED1 4.02 mm to (21.6, 3.81), turned to 180 degrees
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Connections:
- net GND: now also X1.P$1, X1.P$2, X1.P$3, X1.P$4
- net GNDO: now also X2.P$0, X2.P$1
Routing:
- net +5V: track 0.00 -> 108.7 mm
- net GND: track 0.00 -> 90.8 mm, vias 0 -> 8
- net 5VUSB: track 0.00 -> 78.2 mm
- net N$5: track 0.00 -> 67.9 mm
- net D+: track 0.00 -> 51.8 mm, vias 0 -> 1
- net D-: track 0.00 -> 50.7 mm
- net GNDO: track 0.00 -> 45.2 mm
- net N$4: track 0.00 -> 43.6 mm
- net N$3: track 0.00 -> 42.9 mm, vias 0 -> 2
- net 5VESP: track 0.00 -> 42.3 mm
- net DATAON: track 0.00 -> 32.5 mm
- net PWRON: track 0.00 -> 26.4 mm, vias 0 -> 1
- net D+O: track 0.00 -> 22.1 mm
- net VCC0: track 0.00 -> 21.1 mm
- net D-O: track 0.00 -> 21.1 mm
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- added copper zone on layer 1, net GND
- added copper zone on layer 16, net GND
Other:
- board size 100 x 80 mm -> 26.7 x 77.7 mm
- board text added: "EXT"
- board text added: "INT"
- board text added: "PWR SRC"

Commit message: Work work
Parts:
- UIN: device con-lstb:MA05-1 -> USB Switch PCB:FE05-1
- UOUT: device con-lstb:MA04-1 -> USB Switch PCB:FE04-1
- moved UOUT 1.27 mm to (11.4, 62.2)
Routing:
- net GND: vias 8 -> 9
Other:
- board size 26.7 x 77.7 mm -> 26.7 x 77.5 mm
- board text added: "USB Switch 1.0 git.erim.se/hw/usb-switch"

Commit message: More work on switch.
Parts:
- D1, D2: device diode:SOT23 -> USB Switch PCB:SOT23
- moved LED2 2.54 mm to (6.35, 3.81), turned to 0 degrees
- moved LED1 1.27 mm to (20.3, 3.81), turned to 0 degrees
- moved R1 0.64 mm to (22.2, 7.62)
- moved R4 0.64 mm to (24.8, 7.62)
- moved U$1 0.64 mm to (22.2, 55.9)
- moved UIN 0.64 mm to (13.3, 7.62)
- moved X1 0.64 mm to (13.3, 1.27)
- moved X2 0.64 mm to (13.3, 66.0)
- moved R2 0.64 mm to (4.45, 7.62)
- moved U$2 0.64 mm to (4.45, 55.9)
- moved R3 0.64 mm to (1.91, 7.62)
- moved U1 0.64 mm to (1.91, 19.1)
- moved D1 0.63 mm to (15.9, 52.1)
- moved D2 0.63 mm to (10.8, 52.1)
- moved Q1 0.63 mm to (15.9, 47.0)
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Connections:
- net N$16 renamed ID
Routing:
- net +5V: track 108.7 -> 102.9 mm
- net N$2: track 4.77 -> 3.07 mm
- net N$1: track 4.73 -> 3.12 mm
- net GND: vias 9 -> 3

Commit message: Final touches.
Connections:
- removed net 5VESP: S1.S, U1.5V
- net +5V: now also S1.S, U1.5V
Routing:
- net +5V: track 102.9 -> 145.2 mm
- net 5VESP: track 42.3 -> 0.00 mm
- net PWRON: track 26.4 -> 30.3 mm
Changed lines of the file:
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@@
 <via x="17.907" y="20.828" extent="1-16" drill="0.35"/>
 <via x="7.493" y="35.052" extent="1-16" drill="0.35"/>
+<wire x1="9.535" y1="1.27" x2="10.235" y2="3.82" width="0" layer="19" extent="1-1"/>
 </signal>
 <signal name="+5V">
@@
 <wire x1="23.1988" y1="5.6388" x2="20.32" y2="2.76" width="0.1524" layer="1"/>
 <wire x1="25.45005625" y1="5.6388" x2="23.1988" y2="5.6388" width="0.1524" layer="1"/>
+<contactref element="S1" pad="S"/>
+<contactref element="U1" pad="5V"/>
+<wire x1="2.6162" y1="19.05" x2="1.905" y2="19.05" width="0.1524" layer="16"/>
+<wire x1="5.8166" y1="22.2504" x2="2.6162" y2="19.05" width="0.1524" layer="16"/>
+<wire x1="5.8166" y1="51.054" x2="5.8166" y2="22.2504" width="0.1524" layer="16"/>
+<wire x1="10.6934" y1="55.9308" x2="5.8166" y2="51.054" width="0.1524" layer="16"/>
+<wire x1="10.6934" y1="57.15" x2="10.6934" y2="55.9308" width="0.1524" layer="16"/>
+<wire x1="10.6934" y1="57.15" x2="10.795" y2="57.15" width="0.1524" layer="16"/>
+<wire x1="12.065" y1="58.3692" x2="10.795" y2="57.15" width="0" layer="19" extent="1-1"/>
 </signal>
 <signal name="N$1">
@@
 <contactref element="U1" pad="D1"/>
 <contactref element="R3" pad="1"/>
-<wire x1="2.0066" y1="7.1628" x2="2.0066" y2="6.858" width="0.1524" layer="1"/>
+<wire x1="2.0066" y1="6.858" x2="2.0066" y2="7.1628" width="0.1524" layer="1"/>
 <wire x1="3.5306" y1="8.6868" x2="2.0066" y2="7.1628" width="0.1524" layer="1"/>
-<wire x1="3.5306" y1="20.8788" x2="3.5306" y2="8.6868" width="0.1524" layer="1"/>
-<wire x1="3.5306" y1="30.1752" x2="3.5306" y2="20.8788" width="0.1524" layer="16"/>
-<wire x1="2.0066" y1="31.6992" x2="3.5306" y2="30.1752" width="0.1524" layer="16"/>
-<wire x1="2.0066" y1="6.858" x2="1.905" y2="6.77" width="0.1524" layer="1"/>
+<wire x1="1.905" y1="6.77" x2="2.0066" y2="6.858" width="0.1524" layer="1"/>
 <wire x1="2.0066" y1="31.6992" x2="1.905" y2="31.75" width="0.1524" layer="16"/>
-<via x="3.5306" y="20.8788" extent="1-16" drill="0.35"/>
+<via x="4.1656" y="22.7838" extent="1-16" drill="0.35"/>
+<wire x1="1.2563125" y1="22.3726" x2="1.1224" y2="22.2386875" width="0.1524" layer="1"/>
+<wire x1="1.1224" y1="22.2386875" x2="1.1224" y2="20.9413125" width="0.1524" layer="1"/>
+<wire x1="3.7544" y1="22.3726" x2="4.1656" y2="22.7838" width="0.1524" layer="1"/>
+<wire x1="3.7544" y1="22.3726" x2="1.2563125" y2="22.3726" width="0.1524" layer="1"/>
+<wire x1="1.1224" y1="20.9413125" x2="3.5306" y2="18.5331125" width="0.1524" layer="1"/>
+<wire x1="3.5306" y1="18.5331125" x2="3.5306" y2="8.6868" width="0.1524" layer="1"/>
+<wire x1="4.1656" y1="29.5402" x2="4.1656" y2="22.7838" width="0.1524" layer="16"/>
+<wire x1="4.1656" y1="29.5402" x2="2.0066" y2="31.6992" width="0.1524" layer="16"/>
 </signal>
 <signal name="N$3">
@@
 <wire x1="14.0462" y1="3.9624" x2="13.985" y2="3.95" width="0.1524" layer="1"/>
 </signal>
-<signal name="5VESP">
-<contactref element="S1" pad="S"/>
-<contactref element="U1" pad="5V"/>
-<wire x1="2.6162" y1="19.05" x2="1.905" y2="19.05" width="0.1524" layer="16"/>
-<wire x1="5.8166" y1="22.2504" x2="2.6162" y2="19.05" width="0.1524" layer="16"/>
-<wire x1="5.8166" y1="51.054" x2="5.8166" y2="22.2504" width="0.1524" layer="16"/>
-<wire x1="10.6934" y1="55.9308" x2="5.8166" y2="51.054" width="0.1524" layer="16"/>
-<wire x1="10.6934" y1="57.15" x2="10.6934" y2="55.9308" width="0.1524" layer="16"/>
-<wire x1="10.6934" y1="57.15" x2="10.795" y2="57.15" width="0.1524" layer="16"/>
-</signal>
 <signal name="DATAON">

Commit message: I'm gonna start messing shit up soon.
Parts:
- added C1, C4: 100nF, rcl:C0603
- added C2, C3: 10µF, rcl:C0603
- added EXTPWR: (no value), SparkFun-Connectors:1X02
- added MCU: (no value), ESP8266-ESP12E:ESP8266-ESP12E
- added R5, R6: 470Ω, rcl:R0603
- added U$3: CH340G, ch340g:SOIC16
- added UIN1: (no value), USB Switch PCB:FE05-1
- R1: value 330 Ω -> 330Ω
- R3, R4: value 1 kΩ -> 1kΩ
- turned D1 to 180 degrees
- turned D2 to 180 degrees
Connections:
- new net N$10: U$3.5, UIN1.3
- new net N$7: R5.2, U$3.2
- new net N$8: R6.2, U$3.3
- new net N$9: U$3.6, UIN1.2
- new net RXD: MCU.15, R6.1
- new net TXD: MCU.16, R5.1
- net +5V: now also C1.1, C2.1, C3.1, C4.1, EXTPWR.1, MCU.8, U$3.16, U$3.4
- net DATAON: now also MCU.13
- net GND: now also C1.2, C2.2, C3.2, C4.2, EXTPWR.2, MCU.9, U$3.1, UIN1.5
- net PWRON: now also MCU.14
Routing:
- net GND: track 90.8 -> 1.12 mm, vias 3 -> 2
- net +5V: track 145.2 -> 112.4 mm, vias 0 -> 3
- net 5VUSB: track 78.5 -> 62.3 mm, vias 0 -> 1
- net N$5: track 67.9 -> 78.3 mm
- net D-O: track 21.1 -> 28.5 mm
- net N$6: track 12.9 -> 16.1 mm
- net GNDO: track 45.2 -> 43.3 mm
- net PWRON: track 30.3 -> 28.5 mm, vias 1 -> 0
- net D+: track 51.8 -> 50.2 mm, vias 1 -> 0
- net D-: track 50.7 -> 51.4 mm, vias 0 -> 1
- net D+O: track 22.1 -> 21.5 mm
- net VCC0: track 21.1 -> 21.7 mm
Other:
- board text added: "EXT + -"
- board text added: "TODO: Move everything to side-by-side usb. Switch to USB B."
- board text added: "USB Switch 1.1 git.erim.se /hw/usb-switch"
- board text removed: "USB Switch 1.0 git.erim.se/hw/usb-switch"

Commit message: Working on new board revision.
Parts:
- removed R3, R4: 1kΩ, rcl:R0603
- removed U1: D1MINI, USB Switch PCB:D1MINI
- R1: value 330Ω -> 1kΩ
- R2: value 330 Ω -> 1kΩ
Connections:
- removed net DATAON: MCU.13, R4.1, U1.D2
- removed net N$3: Q1.1, R3.2
- removed net N$4: Q2.1, R4.2
- removed net PWRON: MCU.14, R3.1, U1.D1
- new net DATAGATE: MCU.14, Q2.1
- new net POWERGATE: MCU.13, Q1.1
- net +5V: no longer U1.5V
- net GND: no longer U1.GND
Routing:
- net N$4: track 43.7 -> 0.00 mm
- net DATAGATE: track 0.00 -> 43.6 mm
- net N$3: track 42.8 -> 0.00 mm, vias 2 -> 0
- net DATAON: track 32.5 -> 0.00 mm
- net PWRON: track 28.5 -> 0.00 mm
Changed lines of the file:
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@@
 <attribute name="NAME" x="9.271" y="48.006" size="0.635" layer="25" font="vector"/>
 </element>
-<element name="R1" library="rcl" library_urn="urn:adsk.eagle:library:334" package="R0603" value="330Ω" x="22.225" y="7.62" smashed="yes" rot="R270">
+<element name="R1" library="rcl" library_urn="urn:adsk.eagle:library:334" package="R0603" value="1kΩ" x="22.225" y="7.62" smashed="yes" rot="R270">
 <attribute name="NAME" x="21.717" y="9.271" size="0.635" layer="25" font="vector"/>
 </element>
-<element name="R2" library="rcl" library_urn="urn:adsk.eagle:library:334" package="R0603" value="330 Ω" x="4.445" y="7.62" smashed="yes" rot="R90">
+<element name="R2" library="rcl" library_urn="urn:adsk.eagle:library:334" package="R0603" value="1kΩ" x="4.445" y="7.62" smashed="yes" rot="R90">
 <attribute name="NAME" x="5.08" y="9.906" size="0.635" layer="25" font="vector" rot="R180"/>
-</element>
-<element name="R3" library="rcl" library_urn="urn:adsk.eagle:library:334" package="R0603" value="1kΩ" x="1.905" y="7.62" smashed="yes" rot="R90">
-<attribute name="NAME" x="2.54" y="9.906" size="0.635" layer="25" font="vector" rot="R180"/>
-</element>
-<element name="R4" library="rcl" library_urn="urn:adsk.eagle:library:334" package="R0603" value="1kΩ" x="24.765" y="7.62" smashed="yes" rot="R90">
-<attribute name="NAME" x="24.257" y="9.271" size="0.635" layer="25" font="vector"/>
 </element>
 <element name="S1" library="USB Switch PCB" package="SWITCH" value="SWITCH" x="15.875" y="57.15" smashed="yes" rot="R180"/>
 <element name="U$1" library="USB Switch PCB" package="EC2-5NU" value="EC2-5NUEC2-5NU" x="22.225" y="55.88" smashed="yes" rot="R180"/>
 <element name="U$2" library="USB Switch PCB" package="EC2-5NU" value="EC2-5NUEC2-5NU" x="4.445" y="55.88" smashed="yes" rot="R180"/>
-<element name="U1" library="USB Switch PCB" package="D1MINI" value="D1MINI" x="1.905" y="19.05" smashed="yes"/>
 <element name="UIN" library="USB Switch PCB" package="FE05-1" value="" x="13.335" y="7.62" smashed="yes">
 <attribute name="MF" value="" x="13.335" y="7.62" size="1.778" layer="27" display="off"/>
@@
 <contactref element="Q2" pad="2"/>
 <contactref element="R2" pad="2"/>
-<contactref element="U1" pad="GND"/>
 <contactref element="X1" pad="GND"/>
 <contactref element="UIN" pad="5"/>
@@
 <wire x1="12.7" y1="22.86" x2="11.745" y2="45.89" width="0" layer="19" extent="1-1"/>
 <wire x1="6.35" y1="22.86" x2="12.7" y2="22.86" width="0" layer="19" extent="1-1"/>
-<wire x1="1.905" y1="21.59" x2="6.35" y2="22.86" width="0" layer="19" extent="1-1"/>
-<wire x1="4.445" y1="8.47" x2="1.905" y2="21.59" width="0" layer="19" extent="1-1"/>
+<wire x1="4.445" y1="8.47" x2="6.35" y2="22.86" width="0" layer="19" extent="1-1"/>
 <wire x1="10.235" y1="3.82" x2="4.445" y2="8.47" width="0" layer="19" extent="1-1"/>
 <wire x1="9.535" y1="1.27" x2="10.235" y2="3.82" width="0" layer="19" extent="1-1"/>
@@
 <contactref element="D1" pad="3"/>
 <contactref element="S1" pad="S"/>
-<contactref element="U1" pad="5V"/>
 <contactref element="EXTPWR" pad="1"/>
 <wire x1="21.0312" y1="59.7408" x2="19.812" y2="58.5216" width="0.1524" layer="1"/>
@@
 <wire x1="1.9812" y1="19.05" x2="1.9812" y2="18.4404" width="0.1524" layer="16"/>
 <wire x1="6.2484" y1="2.8956" x2="6.35" y2="2.76" width="0.1524" layer="1"/>
-<wire x1="1.9812" y1="19.05" x2="1.905" y2="19.05" width="0.1524" layer="16"/>
 <wire x1="19.2024" y1="2.8956" x2="20.2692" y2="2.8956" width="0.1524" layer="1"/>
 <wire x1="6.4008" y1="2.8956" x2="19.2024" y2="2.8956" width="0.1524" layer="16"/>
@@
 <wire x1="16.9164" y1="53.0352" x2="16.825" y2="53.17" width="0.1524" layer="1"/>
 </signal>
-<signal name="PWRON">
-<contactref element="U1" pad="D1"/>
-<contactref element="R3" pad="1"/>
-<wire x1="1.8288" y1="7.1628" x2="1.8288" y2="6.858" width="0.1524" layer="1"/>
-<wire x1="1.0668" y1="7.9248" x2="1.8288" y2="7.1628" width="0.1524" layer="1"/>
-<wire x1="1.0668" y1="9.144" x2="1.0668" y2="7.9248" width="0.1524" layer="1"/>
-<wire x1="1.6764" y1="9.7536" x2="1.0668" y2="9.144" width="0.1524" layer="1"/>
-<wire x1="1.6764" y1="16.1544" x2="1.6764" y2="9.7536" width="0.1524" layer="1"/>
-<wire x1="3.81" y1="18.288" x2="1.6764" y2="16.1544" width="0.1524" layer="1"/>
-<wire x1="3.81" y1="26.0604" x2="3.81" y2="18.288" width="0.1524" layer="1"/>
-<wire x1="1.6764" y1="28.194" x2="3.81" y2="26.0604" width="0.1524" layer="1"/>
-<wire x1="1.524" y1="28.194" x2="1.6764" y2="28.194" width="0.1524" layer="1"/>
-<wire x1="0.4572" y1="29.2608" x2="1.524" y2="28.194" width="0.1524" layer="1"/>
-<wire x1="0.4572" y1="30.3276" x2="0.4572" y2="29.2608" width="0.1524" layer="1"/>
-<wire x1="1.8288" y1="31.6992" x2="0.4572" y2="30.3276" width="0.1524" layer="1"/>
-<wire x1="1.8288" y1="6.858" x2="1.905" y2="6.77" width="0.1524" layer="1"/>
-<wire x1="1.8288" y1="31.6992" x2="1.905" y2="31.75" width="0.1524" layer="1"/>
-<contactref element="MCU" pad="14"/>
-<wire x1="-13.645" y1="10.095" x2="1.0668" y2="9.144" width="0" layer="19" extent="1-1"/>
-</signal>
-<signal name="N$3">
-<contactref element="Q1" pad="1"/>
-<contactref element="R3" pad="2"/>
-<wire x1="1.9812" y1="16.002" x2="1.9812" y2="8.5344" width="0.1524" layer="1"/>
-<wire x1="8.6868" y1="22.7076" x2="1.9812" y2="16.002" width="0.1524" layer="1"/>
-<wire x1="8.6868" y1="23.0124" x2="8.6868" y2="22.7076" width="0.1524" layer="16"/>
-<wire x1="14.7828" y1="29.1084" x2="8.6868" y2="23.0124" width="0.1524" layer="16"/>
-<wire x1="14.7828" y1="44.6532" x2="14.7828" y2="29.1084" width="0.1524" layer="16"/>
-<wire x1="14.9352" y1="44.8056" x2="14.7828" y2="44.6532" width="0.1524" layer="1"/>
-<wire x1="14.9352" y1="45.8724" x2="14.9352" y2="44.8056" width="0.1524" layer="1"/>
-<wire x1="1.9812" y1="8.5344" x2="1.905" y2="8.47" width="0.1524" layer="1"/>
-<wire x1="14.9352" y1="45.8724" x2="14.925" y2="45.89" width="0.1524" layer="1"/>
-<via x="8.6868" y="22.7076" extent="1-16" drill="0.3048"/>
-<via x="14.7828" y="44.6532" extent="1-16" drill="0.3048"/>
-</signal>
-<signal name="N$4">
-<contactref element="R4" pad="2"/>
+<signal name="DATAGATE">
 <contactref element="Q2" pad="1"/>
 <wire x1="24.8412" y1="15.8496" x2="24.8412" y2="8.5344" width="0.1524" layer="1"/>
 <wire x1="9.906" y1="30.7848" x2="24.8412" y2="15.8496" width="0.1524" layer="1"/>
 <wire x1="9.906" y1="45.8724" x2="9.906" y2="30.7848" width="0.1524" layer="1"/>
-<wire x1="24.8412" y1="8.5344" x2="24.765" y2="8.47" width="0.1524" layer="1"/>
 <wire x1="9.906" y1="45.8724" x2="9.845" y2="45.89" width="0.1524" layer="1"/>
+<contactref element="MCU" pad="14"/>
+<wire x1="-13.645" y1="10.095" x2="9.906" y2="30.7848" width="0" layer="19" extent="1-1"/>
 </signal>
 <signal name="VCC0">
@@
 <wire x1="13.8684" y1="3.9624" x2="13.985" y2="3.95" width="0.1524" layer="1"/>
 <wire x1="15.8496" y1="7.62" x2="15.875" y2="7.62" width="0.1524" layer="1"/>
-</signal>
-<signal name="DATAON">
-<contactref element="U1" pad="D2"/>
-<contactref element="R4" pad="1"/>
-<wire x1="24.6888" y1="7.1628" x2="24.6888" y2="6.858" width="0.1524" layer="1"/>
-<wire x1="23.9268" y1="7.9248" x2="24.6888" y2="7.1628" width="0.1524" layer="1"/>
-<wire x1="23.9268" y1="8.0772" x2="23.9268" y2="7.9248" width="0.1524" layer="1"/>
-<wire x1="23.0124" y1="8.9916" x2="23.9268" y2="8.0772" width="0.1524" layer="1"/>
-<wire x1="23.0124" y1="9.144" x2="23.0124" y2="8.9916" width="0.1524" layer="1"/>
-<wire x1="3.81" y1="28.3464" x2="23.0124" y2="9.144" width="0.1524" layer="1"/>
-<wire x1="3.3528" y1="28.3464" x2="3.81" y2="28.3464" width="0.1524" layer="1"/>
-<wire x1="2.8956" y1="28.8036" x2="3.3528" y2="28.3464" width="0.1524" layer="1"/>
-<wire x1="2.7432" y1="28.8036" x2="2.8956" y2="28.8036" width="0.1524" layer="1"/>
-<wire x1="2.4384" y1="29.1084" x2="2.7432" y2="28.8036" width="0.1524" layer="1"/>
-<wire x1="1.9812" y1="29.1084" x2="2.4384" y2="29.1084" width="0.1524" layer="1"/>
-<wire x1="24.6888" y1="6.858" x2="24.765" y2="6.77" width="0.1524" layer="1"/>
-<wire x1="1.9812" y1="29.1084" x2="1.905" y2="29.21" width="0.1524" layer="1"/>
-<contactref element="MCU" pad="13"/>
-<wire x1="-13.645" y1="8.095" x2="1.9812" y2="29.1084" width="0" layer="19" extent="1-1"/>
 </signal>
 <signal name="N$5">
@@
 <wire x1="-25.4" y1="-14.125" x2="-20.955" y2="-52.705" width="0" layer="19" extent="1-1"/>
 </signal>
+<signal name="POWERGATE">
+<contactref element="Q1" pad="1"/>
+<contactref element="MCU" pad="13"/>
+<wire x1="-13.645" y1="8.095" x2="14.925" y2="45.89" width="0" layer="19" extent="1-1"/>
+</signal>
 </signals>

Commit message: More work, looks like shit now.
Parts:
- removed UIN1: (no value), USB Switch PCB:FE05-1
- added C5, C6: 20pF, rcl:C0603
- added C7: 100nF, rcl:C0603
- added C8, C9: 1µF, rcl:C0603
- added D3: BAS21LT1, USB Switch PCB:SOT23
- added Q3: 12 MHz, USB Switch PCB:CSM-3X
- added R3, R4: 12kΩ, rcl:R0603
- added U$4: UMH3N, USB Switch PCB:SOT363
- added U$5: MIC5504-3.3YM5SOT23, USB Switch PCB:SOT-23-5
- added X3: AMPHENOL-0001LF, USB Switch PCB:10118192-0001LF
- moved R6 76.5 mm to (17.7, 34.8), flipped to the bottom
- moved R5 74.1 mm to (17.7, 36.7), flipped to the bottom
- moved C4 69.7 mm to (4.63, 17.0), flipped to the bottom, turned to 180 degrees
- moved C2 66.4 mm to (1.91, 25.0), flipped to the bottom, turned to 270 degrees
- moved C3 62.1 mm to (2.29, 14.7), flipped to the bottom, turned to 270 degrees
- moved C1 59.4 mm to (2.16, 20.4), flipped to the bottom, turned to 270 degrees
- moved U$3 41.6 mm to (6.48, 14.5)
- moved MCU 38.7 mm to (9.14, 30.9)
- moved D2 7.47 mm to (4.45, 56.0), flipped to the bottom
- moved Q2 7.47 mm to (4.45, 50.9), flipped to the bottom, turned to 180 degrees
- moved D1 7.44 mm to (22.2, 56.0), flipped to the bottom
- moved Q1 7.26 mm to (22.1, 50.7), flipped to the bottom, turned to 180 degrees
- moved R1 4.24 mm to (20.3, 3.84), flipped to the bottom, turned to 90 degrees
- moved R2 4.12 mm to (6.35, 3.97), flipped to the bottom, turned to 270 degrees
Connections:
- net 5VUSB renamed VCCI
- net D+ renamed D+I
- net D- renamed D-I
- net N$5 renamed DATACOIL
- net N$6 renamed POWERCOIL
- net VCC0 renamed VCCO
- removed net N$10: U$3.5, UIN1.3
- removed net N$9: U$3.6, UIN1.2
- new net D+ESP: U$3.5, X3.D+
- new net D-ESP: U$3.6, X3.D-
- new net DTR: U$3.13, U$4.2, U$4.4
- new net EN: MCU.3, R4.2
- new net GPIO0: MCU.12, U$4.3
- new net N$4: D3.1, X3.VCC
- new net RST: C7.1, MCU.1, R3.2, U$4.6
- new net RTS: U$3.14, U$4.1, U$4.5
- new net XI: C6.1, Q3.P$2, U$3.7
- new net XO: C5.1, Q3.P$1, U$3.8
- net +5V: now also C8.1, C9.1, D3.3, R3.1, R4.1, U$5.1, U$5.3, U$5.5
- net GND: now also C5.2, C6.2, C7.2, C8.2, C9.2, U$5.2, X3.GND, X3.P$1, X3.P$2, X3.P$3, X3.P$4; no longer UIN1.5
Routing:
- net +5V: track 112.3 -> 0.00 mm, vias 3 -> 0
- net DATACOIL: track 78.3 -> 0.00 mm
- net VCCI: track 62.3 -> 0.00 mm, vias 1 -> 0
- net D-I: track 51.4 -> 0.00 mm, vias 1 -> 0
- net D+I: track 50.2 -> 0.00 mm
- net DATAGATE: track 43.6 -> 0.00 mm
- net GNDO: track 43.3 -> 0.00 mm
- net D-O: track 28.5 -> 0.00 mm
- net VCCO: track 21.7 -> 0.00 mm
- net D+O: track 21.5 -> 0.00 mm
- net POWERCOIL: track 16.1 -> 0.00 mm
- net ID: track 4.93 -> 0.00 mm
- net N$2: track 3.50 -> 0.00 mm
- net N$1: track 3.50 -> 0.00 mm
- net GND: track 1.12 -> 0.00 mm, vias 2 -> 0
- removed copper zone on layer 1, net GND
- removed copper zone on layer 16, net GND
Other:
- board size 26.7 x 77.5 mm -> 27.1 x 100 mm
- board text removed: "TODO: Move everything to side-by-side usb. Switch to USB B."

Commit message: Total redesign of, well, everything.
Parts:
- moved R3 102.5 mm to (0.22, 90.6), flipped to the bottom
- moved C7 99.3 mm to (-3.81, 90.6), flipped to the bottom
- moved UIN 87.4 mm to (-37.5, 78.7)
- moved X1 87.4 mm to (-37.5, 72.4)
- moved LED1 87.0 mm to (-30.7, 74.3)
- moved R1 87.0 mm to (-30.8, 74.3)
- moved LED2 86.7 mm to (-44.1, 74.3)
- moved R2 86.7 mm to (-44.1, 74.5)
- moved C3 78.4 mm to (14.5, 92.1), turned to 90 degrees
- moved U$4 77.4 mm to (-7.30, 89.9), turned to 270 degrees
- moved C4 76.0 mm to (16.5, 92.1), turned to 90 degrees
- moved R4 72.0 mm to (-10.5, 86.8), turned to 180 degrees
- moved C5 72.0 mm to (19.8, 83.7)
- moved C6 72.0 mm to (19.8, 89.1)
- moved Q3 72.0 mm to (19.8, 86.4)
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Connections:
- new net +3V3: C3.1, C4.1, C8.1, U$3.16, U$5.5
- net +5V: no longer C3.1, C4.1, C8.1, U$3.16, U$5.5
Other:
- board outline removed
