File: pcb/USB Switch PCB.sch (EAGLE design)
At the start: 18 parts, among them Q1 2N7002P, Q2 2N7002P, U1 D1MINI, X1 AMPHENOL-0001LF, X2 UE27-USBA

Commit message: Auto-routed PCB with lots of nice stuff.
Parts:
- LED1: value GREEN -> ACT
- LED2: value RED -> PWR
Changed lines of the file:
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@@
 </classes>
 <parts>
-<part name="LED1" library="led" library_urn="urn:adsk.eagle:library:259" deviceset="LED" device="CHIPLED_0805" value="GREEN"/>
-<part name="LED2" library="led" library_urn="urn:adsk.eagle:library:259" deviceset="LED" device="CHIPLED_0805" value="RED"/>
+<part name="LED1" library="led" library_urn="urn:adsk.eagle:library:259" deviceset="LED" device="CHIPLED_0805" value="ACT"/>
+<part name="LED2" library="led" library_urn="urn:adsk.eagle:library:259" deviceset="LED" device="CHIPLED_0805" value="PWR"/>
 <part name="R1" library="rcl" library_urn="urn:adsk.eagle:library:334" deviceset="R-EU_" device="R0603" value="330 Ω"/>
 <part name="R2" library="rcl" library_urn="urn:adsk.eagle:library:334" deviceset="R-EU_" device="R0603" value="330 Ω"/>

Commit message: Work work
Parts:
- UIN: device con-lstb:MA05-1 -> USB Switch PCB:FE05-1
- UOUT: device con-lstb:MA04-1 -> USB Switch PCB:FE04-1
Changed lines of the file:
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@@
 <part name="X1" library="USB Switch PCB" deviceset="AMPHENOL-0001LF" device=""/>
 <part name="X2" library="USB Switch PCB" deviceset="UE27-USBA" device=""/>
-<part name="UOUT" library="con-lstb" library_urn="urn:adsk.eagle:library:162" deviceset="MA04-1" device=""/>
-<part name="UIN" library="con-lstb" library_urn="urn:adsk.eagle:library:162" deviceset="MA05-1" device=""/>
+<part name="UIN" library="USB Switch PCB" deviceset="FE05-1" device=""/>
+<part name="UOUT" library="USB Switch PCB" deviceset="FE04-1" device=""/>
 </parts>
 <sheets>
@@
 <instance part="X1" gate="G$1" x="-38.1" y="83.82"/>
 <instance part="X2" gate="G$1" x="-30.48" y="66.04"/>
-<instance part="UOUT" gate="1" x="-48.26" y="71.12"/>
 <instance part="UIN" gate="G$1" x="-53.34" y="88.9"/>
+<instance part="UOUT" gate="G$1" x="-48.26" y="71.12"/>
 </instances>
 <busses>
@@
 <pinref part="U$1" gate="G$1" pin="A1"/>
 <pinref part="X2" gate="G$1" pin="VCC"/>
-<pinref part="UOUT" gate="1" pin="1"/>
 <wire x1="-40.64" y1="66.04" x2="-27.94" y2="66.04" width="0.1524" layer="91"/>
 <junction x="-27.94" y="66.04"/>
+<pinref part="UOUT" gate="G$1" pin="1"/>
 </segment>
 </net>
@@
 <wire x1="2.54" y1="73.66" x2="2.54" y2="66.04" width="0.1524" layer="91"/>
 <pinref part="X2" gate="G$1" pin="GND"/>
-<pinref part="UOUT" gate="1" pin="4"/>
 <wire x1="-40.64" y1="73.66" x2="-27.94" y2="73.66" width="0.1524" layer="91"/>
 <junction x="-27.94" y="73.66"/>
+<pinref part="UOUT" gate="G$1" pin="4"/>
 </segment>
 </net>
@@
 <segment>
 <pinref part="X2" gate="G$1" pin="D-"/>
-<pinref part="UOUT" gate="1" pin="2"/>
 <wire x1="-40.64" y1="68.58" x2="-27.94" y2="68.58" width="0.1524" layer="91"/>
 <pinref part="U$2" gate="G$1" pin="A1"/>
@@
 <wire x1="-22.86" y1="68.58" x2="-27.94" y2="68.58" width="0.1524" layer="91"/>
 <junction x="-27.94" y="68.58"/>
+<pinref part="UOUT" gate="G$1" pin="2"/>
 </segment>
 </net>
@@
 <segment>
 <pinref part="X2" gate="G$1" pin="D+"/>
-<pinref part="UOUT" gate="1" pin="3"/>
 <wire x1="-40.64" y1="71.12" x2="-27.94" y2="71.12" width="0.1524" layer="91"/>
 <pinref part="U$2" gate="G$1" pin="A2"/>
@@
 <wire x1="-20.32" y1="71.12" x2="-27.94" y2="71.12" width="0.1524" layer="91"/>
 <junction x="-27.94" y="71.12"/>
+<pinref part="UOUT" gate="G$1" pin="3"/>
 </segment>
 </net>

Commit message: More work on switch.
Parts:
- D1, D2: device diode:BAS40 -> USB Switch PCB:BAS40
Connections:
- net N$16 renamed ID
Changed lines of the file:
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@@
 <part name="R3" library="rcl" library_urn="urn:adsk.eagle:library:334" deviceset="R-EU_" device="R0603" value="1 kΩ"/>
 <part name="R4" library="rcl" library_urn="urn:adsk.eagle:library:334" deviceset="R-EU_" device="R0603" value="1 kΩ"/>
-<part name="D1" library="diode" library_urn="urn:adsk.eagle:library:210" deviceset="BAS40" device="" value="BAS21LT1"/>
+<part name="D1" library="USB Switch PCB" deviceset="BAS40" device="" value="BAS21LT1"/>
 <part name="Q1" library="USB Switch PCB" deviceset="2N7002P" device="2N7002P" value="2N7002P"/>
 <part name="Q2" library="USB Switch PCB" deviceset="2N7002P" device="2N7002P" value="2N7002P"/>
-<part name="D2" library="diode" library_urn="urn:adsk.eagle:library:210" deviceset="BAS40" device="" value="BAS21LT1"/>
+<part name="D2" library="USB Switch PCB" deviceset="BAS40" device="" value="BAS21LT1"/>
 <part name="GND3" library="supply1" library_urn="urn:adsk.eagle:library:371" deviceset="GND" device=""/>
 <part name="GND4" library="supply1" library_urn="urn:adsk.eagle:library:371" deviceset="GND" device=""/>
@@
 </segment>
 </net>
-<net name="N$16" class="0">
+<net name="ID" class="0">
 <segment>
 <pinref part="UIN" gate="G$1" pin="4"/>
@@
 </sheet>
 </sheets>
+<errors>
+</errors>
 </schematic>
 </drawing>

Commit message: Final touches.
Connections:
- removed net 5VESP: S1.S, U1.5V
- net +5V: now also S1.S, U1.5V
Changed lines of the file:
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@@
 <part name="UIN" library="USB Switch PCB" deviceset="FE05-1" device=""/>
 <part name="UOUT" library="USB Switch PCB" deviceset="FE04-1" device=""/>
+<part name="P+4" library="supply1" library_urn="urn:adsk.eagle:library:371" deviceset="+5V" device=""/>
 </parts>
 <sheets>
@@
 <instance part="UIN" gate="G$1" x="-53.34" y="88.9"/>
 <instance part="UOUT" gate="G$1" x="-48.26" y="71.12"/>
+<instance part="P+4" gate="1" x="-55.88" y="53.34"/>
 </instances>
 <busses>
@@
 <wire x1="-12.7" y1="50.8" x2="-12.7" y2="55.88" width="0.1524" layer="91"/>
 <junction x="-12.7" y="55.88"/>
+</segment>
+<segment>
+<pinref part="S1" gate="G$1" pin="S"/>
+<wire x1="-40.64" y1="53.34" x2="-40.64" y2="50.8" width="0.1524" layer="91"/>
+<pinref part="U1" gate="G$1" pin="5V"/>
+<wire x1="-55.88" y1="22.86" x2="-48.26" y2="22.86" width="0.1524" layer="91"/>
+<wire x1="-40.64" y1="50.8" x2="-55.88" y2="50.8" width="0.1524" layer="91"/>
+<wire x1="-55.88" y1="50.8" x2="-55.88" y2="22.86" width="0.1524" layer="91"/>
+<pinref part="P+4" gate="1" pin="+5V"/>
+<junction x="-55.88" y="50.8"/>
 </segment>
 </net>
@@
 </segment>
 </net>
-<net name="5VESP" class="0">
-<segment>
-<pinref part="S1" gate="G$1" pin="S"/>
-<wire x1="-40.64" y1="53.34" x2="-40.64" y2="50.8" width="0.1524" layer="91"/>
-<pinref part="U1" gate="G$1" pin="5V"/>
-<wire x1="-55.88" y1="22.86" x2="-48.26" y2="22.86" width="0.1524" layer="91"/>
-<wire x1="-40.64" y1="50.8" x2="-55.88" y2="50.8" width="0.1524" layer="91"/>
-<wire x1="-55.88" y1="50.8" x2="-55.88" y2="22.86" width="0.1524" layer="91"/>
-</segment>
-</net>

Commit message: I'm gonna start messing shit up soon.
Parts:
- added C1, C4: 100nF, rcl:C-EUC0603
- added C2, C3: 10µF, rcl:C-EUC0603
- added EXTPWR: (no value), SparkFun-Connectors:CONN_02
- added MCU: (no value), ESP8266-ESP12E:ESP8266-12EESP8266-ESP12E
- added R5, R6: 470Ω, rcl:R-EU_R0603
- added U$3: CH340G, ch340g:CH340G
- added UIN1: (no value), USB Switch PCB:FE05-1
- R1: value 330 Ω -> 330Ω
- R3, R4: value 1 kΩ -> 1kΩ
Connections:
- new net N$10: U$3.D+, UIN1.3
- new net N$7: R5.2, U$3.TX
- new net N$8: R6.2, U$3.RX
- new net N$9: U$3.D-, UIN1.2
- new net RXD: MCU.RXD, R6.1
- new net TXD: MCU.TXD, R5.1
- net +5V: now also C1.1, C2.1, C3.1, C4.1, EXTPWR.1, MCU.VCC, U$3.V3, U$3.VCC
- net DATAON: now also MCU.GPIO4
- net GND: now also C1.2, C2.2, C3.2, C4.2, EXTPWR.2, MCU.GND, U$3.GND, UIN1.5
- net PWRON: now also MCU.GPIO5
Other:
- note added: "TODO: Switch to USB B Add external ADC and GPIO Add reset circuit Add 3v3 regulator Add weird UMH3N circuit"

Commit message: Working on new board revision.
Parts:
- removed R3, R4: 1kΩ, rcl:R-EU_R0603
- removed U1: D1MINI, USB Switch PCB:D1MINI
- R1: value 330Ω -> 1kΩ
- R2: value 330 Ω -> 1kΩ
Connections:
- removed net DATAON: MCU.GPIO4, R4.1, U1.D2
- removed net N$3: Q1.G, R3.2
- removed net N$4: Q2.G, R4.2
- removed net PWRON: MCU.GPIO5, R3.1, U1.D1
- new net DATAGATE: MCU.GPIO5, Q2.G
- new net POWERGATE: MCU.GPIO4, Q1.G
- net +5V: no longer U1.5V
- net GND: no longer U1.GND
Other:
- moved on the sheet: C3, C4, LED2, R2, R5, R6, UIN1

Commit message: More work, looks like shit now.
Parts:
- removed UIN1: (no value), USB Switch PCB:FE05-1
- added C5, C6: 20pF, rcl:C-EUC0603
- added C7: 100nF, rcl:C-EUC0603
- added C8, C9: 1µF, rcl:C-EUC0603
- added D3: BAS21LT1, USB Switch PCB:BAS40
- added Q3: 12 MHz, USB Switch PCB:CSM-3XCSM-3X
- added R3, R4: 12kΩ, rcl:R-EU_R0603
- added U$4: UMH3N, USB Switch PCB:UMH3N
- added U$5: MIC5504-3.3YM5SOT23, USB Switch PCB:MIC5504-3.3YM5SOT23
- added X3: AMPHENOL-0001LF, USB Switch PCB:AMPHENOL-0001LF
Connections:
- net 5VUSB renamed VCCI
- net D+ renamed D+I
- net D- renamed D-I
- net N$5 renamed DATACOIL
- net N$6 renamed POWERCOIL
- net VCC0 renamed VCCO
- removed net N$10: U$3.D+, UIN1.3
- removed net N$9: U$3.D-, UIN1.2
- new net D+ESP: U$3.D+, X3.D+
- new net D-ESP: U$3.D-, X3.D-
- new net DTR: U$3.DTR, U$4.BA, U$4.EB
- new net EN: MCU.CH_PD, R4.2
- new net GPIO0: MCU.GPIO0, U$4.CB
- new net N$4: D3.A, X3.VCC
- new net RST: C7.1, MCU.REST, R3.2, U$4.CA
- new net RTS: U$3.RTS, U$4.BB, U$4.EA
- new net XI: C6.1, Q3.2, U$3.XI
- new net XO: C5.1, Q3.1, U$3.XO
- net +5V: now also C8.1, C9.1, D3.C, R3.1, R4.1, U$5.EN, U$5.VIN, U$5.VOUT
- net GND: now also C5.2, C6.2, C7.2, C8.2, C9.2, U$5.GND, X3.GND; no longer UIN1.5
Other:
- note added: "Connectors"
- note added: "ESP12E"
- note added: "Power Management"
- note added: "Relays & Drivers"
- note added: "User Interface"
- moved on the sheet: C1, C2, C3, C4, D1, D2, EXTPWR, LED1, LED2, MCU, Q1, Q2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

Commit message: Total redesign of, well, everything.
Connections:
- new net +3V3: C3.1, C4.1, C8.1, U$3.VCC, U$5.VOUT
- net +5V: no longer C3.1, C4.1, C8.1, U$3.VCC, U$5.VOUT
